File: duckboard/DuckControlBoard/duckboardAI.kicad_pcb (KiCad board)
At the start: 2 copper layers, 154.2 x 127.5 mm, 64 parts, among them J1 BATTERY, J10 Tank Level, J11 5V OUT, J12 PUMP_CONTROL, J14 DOOR_OPEN_LIMIT, J15 DOOR_CLOSE_LIMIT, J16 LIFT_CLOSE_LIMIT, J17PhotoSensor1 Conn_01x02, J2 5V BUCK, J3 LIFT BTS7960, J4 DOOR BTS7960, J6 LIFT CLOSE, J7 LIFT OPEN, J8 DOOR CLOSE, J9 DOOR OPEN, P1 R_Potentiometer, P2 R_Potentiometer, Q1 27P04, Q2 30N06L, U1 ESP32-DevKitC

Commit message: schematic and board work
Parts:
- C1, C10, C11, C12, C13, C14, C2, C3, C5, C6, C7, C8, C9, R1, R10, R11, R12, R13, R14, R15, R17, R18, R19, R2, R20, R21, R22, R23, R25, R26, R4, R5, R6, R7, R8, R9: moved to B.Cu
- J10, J11, J14, J15, J16, J6, J7, J8, J9: footprint Connector_JST:JST_EH_B2B-EH-A_1x02_P2.50mm_Vertical -> Connector_JST:JST_EH_S2B-EH_1x02_P2.50mm_Horizontal
- moved D1 88.3 mm to (177.7, 90.5)
- moved J15 80.3 mm to (168.5, 127.5), turned to 180 degrees
- moved J14 80.0 mm to (183.0, 127.5), turned to 180 degrees
- moved J16 79.7 mm to (153.0, 127.5), turned to 180 degrees
- moved R6 72.0 mm to (185.5, 126.2), turned to 90 degrees
- moved C7 70.2 mm to (160.6, 126.0), turned to 180 degrees
- moved R8 69.1 mm to (148.0, 126.2), turned to -90 degrees
- moved R7 66.7 mm to (163.5, 126.8), turned to -90 degrees
- moved C8 65.2 mm to (145.6, 125.0), turned to 180 degrees
- moved R9 64.5 mm to (178.5, 123.5), turned to -90 degrees
- moved R16 63.2 mm to (177.5, 97.0)
- moved R20 58.9 mm to (145.7, 123.0), turned to 180 degrees
- moved R19 57.3 mm to (160.7, 123.5), turned to 180 degrees
- moved R18 55.1 mm to (163.5, 97.2), turned to -90 degrees
- moved C6 48.5 mm to (181.0, 123.5), turned to -90 degrees
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Other:
- board size 154.2 x 127.5 mm -> 103 x 126.7 mm

Commit message: boarded
Parts:
- added D3: D, Diode_SMD:D_0805_2012Metric, B.Cu at (141.5, 61.6)
- J3, J4: footprint Connector_PinHeader_2.54mm:PinHeader_1x05_P2.54mm_Vertical -> Connector_JST:JST_EH_B5B-EH-A_1x05_P2.50mm_Vertical
- R3: moved to B.Cu
- moved F1 23.8 mm to (122.5, 88.0), turned to 90 degrees
- moved R17 11.9 mm to (131.3, 87.5), turned to 180 degrees
- moved R18 9.97 mm to (161.8, 107.0), turned to 0 degrees
- moved R3 7.59 mm to (206.5, 120.3), turned to -90 degrees
- moved Hole4 6.08 mm to (120.5, 130.0)
- moved Hole3 4.27 mm to (213.0, 130.0)
- moved R16 4.04 mm to (180.0, 93.8), turned to -90 degrees
- moved R12 4.03 mm to (198.2, 56.0)
- moved R15 4.00 mm to (162.2, 56.5)
- moved R13 3.00 mm to (185.7, 56.0)
- moved R14 3.00 mm to (173.7, 56.0)
- moved C5 2.55 mm to (129.1, 100.5)
- moved Hole2 2.24 mm to (213.5, 52.0)
- moved C1 2.04 mm to (121.5, 94.0)
- moved R4 1.85 mm to (127.2, 87.5), turned to 0 degrees
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- renumbered REF** to Hole2, REF** to Hole3, REF** to Hole4, REF** to hole1
Connections:
- C1 pad 1: Net-(C1-Pad1) -> /VBAT_FUSED
- C2 pad 1: Net-(C1-Pad1) -> /VBAT_FUSED
- C3 pad 1: Net-(C1-Pad1) -> /VBAT_FUSED
- F1 pad 1: Net-(C1-Pad1) -> /VBAT_FUSED
- R4 pad 1: /VBAT -> /VBAT_FUSED
- U1 pad 1: unconnected-(U1-3V3-Pad1) -> /+3V3
- U1 pad 2: /GPIO36 -> unconnected-(U1-EN-Pad2)
- U1 pad 3: unconnected-(U1-EN-Pad3) -> /GPIO36
Routing:
- net /GND: track 0.00 -> 246.2 mm, vias 0 -> 10
- net /+3V3: track 0.00 -> 187.6 mm, vias 0 -> 9
- net /MOTOR_CTRL_5V: track 0.00 -> 121.4 mm, vias 0 -> 3
- net /GPIO13: track 0.00 -> 110.1 mm, vias 0 -> 2
- net /GPIO36: track 0.00 -> 110.0 mm, vias 0 -> 3
- net /GPIO12: track 0.00 -> 103.6 mm, vias 0 -> 3
- net /GPIO14: track 0.00 -> 102.8 mm, vias 0 -> 2
- net /+5V: track 0.00 -> 96.8 mm, vias 0 -> 1
- net /GPIO33: track 0.00 -> 87.7 mm, vias 0 -> 4
- net /GPIO34: track 0.00 -> 82.3 mm, vias 0 -> 3
- net /GPIO35: track 0.00 -> 74.4 mm, vias 0 -> 1
- net Net-(U1-GPIO23): track 0.00 -> 71.2 mm, vias 0 -> 1
- net /GPIO17: track 0.00 -> 69.5 mm, vias 0 -> 1
- net /GPIO39: track 0.00 -> 66.5 mm, vias 0 -> 2
- net /GPIO21: track 0.00 -> 64.2 mm, vias 0 -> 3
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- added copper zone on B.Cu, net /GND
Other:
- board size 103 x 126.7 mm -> 103 x 88.2 mm
