File: duckboard/DuckControlBoard/duckboardAI.kicad_sch (KiCad schematic)
At the start: 61 parts, among them J1 BATTERY, J11 5V OUT, J12 12V OUT, J14 Conn_01x02, J15 Conn_01x02, J16 Conn_01x02, J17PhotoSensor1 Conn_01x02, J2 5V BUCK, J3 LIFT BTS7960, J4 DOOR BTS7960, J6 LIFT CLOSE, J7 LIFT OPEN, J8 DOOR CLOSE, J9 DOOR OPEN, P1 R_Potentiometer, P2 R_Potentiometer, Q1 27P04, Q2 30N06L, Q3 30N06L, Q4 27P04, U1 ESP32-DevKitC

Commit message: more board changes
Parts:
- removed Q3: 30N06L, symbol Transistor_FET:Q_NMOS_GSD
- removed Q4: 27P04, symbol Transistor_FET:Q_PMOS_GSD
- removed R24: 10k, symbol Device:R
- added D3: D, symbol Device:D
- added J10: Tank Level, Connector_JST:JST_EH_B2B-EH-A_1x02_P2.50mm_Vertical, symbol Connector_Generic:Conn_01x02
- added R23: 10k, Resistor_SMD:R_0603_1608Metric, symbol Device:R
- C1, C10, C11, C12, C13, C14, C2, C3, C6, C7, C8, C9: footprint (none) -> Capacitor_SMD:C_0805_2012Metric
- C5: value TBD -> 100 nF; footprint (none) -> Capacitor_SMD:C_0805_2012Metric
- D1: footprint (none) -> LED_SMD:LED_Everlight-SMD3528_3.5x2.8mm_67-21ST
- F1: footprint (none) -> Fuse:Fuseholder_Cylinder-5x20mm_Schurter_0031_8201_Horizontal_Open
- J1, J17PhotoSensor1: footprint (none) -> TerminalBlock:TerminalBlock_MaiXu_MX126-5.0-02P_1x02_P5.00mm
- J11, J6, J7, J8, J9: footprint (none) -> Connector_JST:JST_EH_B2B-EH-A_1x02_P2.50mm_Vertical
- J12: value 12V OUT -> PUMP_CONTROL; footprint (none) -> TerminalBlock:TerminalBlock_MaiXu_MX126-5.0-02P_1x02_P5.00mm
- J14: value Conn_01x02 -> DOOR_OPEN_LIMIT; footprint (none) -> Connector_JST:JST_EH_B2B-EH-A_1x02_P2.50mm_Vertical
- J15: value Conn_01x02 -> DOOR_CLOSE_LIMIT; footprint (none) -> Connector_JST:JST_EH_B2B-EH-A_1x02_P2.50mm_Vertical
- J16: value Conn_01x02 -> LIFT_CLOSE_LIMIT; footprint (none) -> Connector_JST:JST_EH_B2B-EH-A_1x02_P2.50mm_Vertical
- J2: footprint (none) -> Connector_PinHeader_2.54mm:PinHeader_1x04_P2.54mm_Vertical
- J3, J4: footprint (none) -> Connector_PinHeader_2.54mm:PinHeader_1x05_P2.54mm_Vertical
- P1: footprint Package_TO_SOT_SMD:SOT-23-8 -> Potentiometer_THT:Potentiometer_Piher_T-16L_Single_Vertical_Hole
- P2: footprint (none) -> Potentiometer_THT:Potentiometer_Piher_T-16L_Single_Vertical_Hole
- Q1, Q2: footprint (none) -> Package_TO_SOT_THT:TO-220-3_Horizontal_TabUp
- R1, R10, R11, R12, R13, R14, R15, R17, R18, R19, R2, R20, R21, R22, R26, R3, R4, R5, R6, R7, R8, R9: footprint (none) -> Resistor_SMD:R_0603_1608Metric
- R16: value 330R -> 120R; footprint (none) -> Resistor_SMD:R_0603_1608Metric
- R25: value 10k -> 470; footprint (none) -> Resistor_SMD:R_0603_1608Metric
- U1: footprint DuckHouse:ESP32-DevKitC -> dLibrary:ESP32-DevKitC
Connections:
- net +3V3: no longer U1.1 (3V3)
- net GND: now also D1.1 (K), D3.1 (K), J10.2 (Pin_2); no longer D1.2 (A)
- net GPIO27: now also R25.1
- net LED_A: now also D1.2 (A), R16.1
- net Tank Level Input: now also R25.2, D3.2 (A), J10.1 (Pin_1); no longer U1.10 (GPIO26)
- net VBAT: now also F1.2, J1.1 (Pin_1); no longer C1.1, C2.1, C3.1, F1.1, J2.3 (Pin_3), R25.1, R26.1
- net at U1.37 (GPIO23): now also R23.2
- net PUMP_CTRL_12V renamed PUMP_CTR
- net PUMP_CTR: now also R23.1
- new net: C1.1, C2.1, C3.1, F1.1
- new net VBAT_FUSED: J2.3 (Pin_3), R26.1
- no-connect marks 0 -> 11
Other:
- note added: "Lift LPWM"
- note added: "Lift RPWM"
- note removed: "4. LIMIT SWITCHES"
- note removed: "Actuator motor power bypasses PCB fuse: battery -> external fuse -> BTS7960 motor controller -> actuator."
- note removed: "Battery divider (R4/R5/C5/R17) is built out in Section 9, right side of sheet. Divider ratio approx 21:1."
- note removed: "Each button: NO to +3V3; 10k external pulldown + 100nF GPIO-to-GND. Signals: J6 GPIO34, J7 GPIO35, J8 GPIO18, J9 GPIO22."
- note removed: "Photosensor (J10) and travel pots (P1/P2) are built out in Section 9, right side of sheet."
- note removed: "and GPIO23/26/27 are simply unused by this design. All 3x GND pins and 3V3/5V are tied to the board GND/+3V3/+5V rails."
- moved on the sheet: C10, C11, C12, C13, C14, C5, C6, C7, C8, C9, D1, J11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

Commit message: schematic and board work
Parts:
- J10, J11, J14, J15, J16, J6, J7, J8, J9: footprint Connector_JST:JST_EH_B2B-EH-A_1x02_P2.50mm_Vertical -> Connector_JST:JST_EH_S2B-EH_1x02_P2.50mm_Horizontal
Changed lines of the file:
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@@
 			)
 		)
-		(property "Footprint" "Connector_JST:JST_EH_B2B-EH-A_1x02_P2.50mm_Vertical"
+		(property "Footprint" "Connector_JST:JST_EH_S2B-EH_1x02_P2.50mm_Horizontal"
 			(at 132.08 115.57 0)
 			(hide yes)
@@
 			)
 		)
-		(property "Footprint" "Connector_JST:JST_EH_B2B-EH-A_1x02_P2.50mm_Vertical"
+		(property "Footprint" "Connector_JST:JST_EH_S2B-EH_1x02_P2.50mm_Horizontal"
 			(at 322.58 116.84 0)
 			(hide yes)
@@
 			)
 		)
-		(property "Footprint" "Connector_JST:JST_EH_B2B-EH-A_1x02_P2.50mm_Vertical"
+		(property "Footprint" "Connector_JST:JST_EH_S2B-EH_1x02_P2.50mm_Horizontal"
 			(at 388.62 163.83 0)
 			(hide yes)
@@
 			)
 		)
-		(property "Footprint" "Connector_JST:JST_EH_B2B-EH-A_1x02_P2.50mm_Vertical"
+		(property "Footprint" "Connector_JST:JST_EH_S2B-EH_1x02_P2.50mm_Horizontal"
 			(at 83.82 130.81 0)
 			(hide yes)
@@
 			)
 		)
-		(property "Footprint" "Connector_JST:JST_EH_B2B-EH-A_1x02_P2.50mm_Vertical"
+		(property "Footprint" "Connector_JST:JST_EH_S2B-EH_1x02_P2.50mm_Horizontal"
 			(at 354.33 104.14 0)
 			(hide yes)
@@
 			)
 		)
-		(property "Footprint" "Connector_JST:JST_EH_B2B-EH-A_1x02_P2.50mm_Vertical"
+		(property "Footprint" "Connector_JST:JST_EH_S2B-EH_1x02_P2.50mm_Horizontal"
 			(at 95.25 194.31 0)
 			(hide yes)
@@
 			)
 		)
-		(property "Footprint" "Connector_JST:JST_EH_B2B-EH-A_1x02_P2.50mm_Vertical"
+		(property "Footprint" "Connector_JST:JST_EH_S2B-EH_1x02_P2.50mm_Horizontal"
 			(at 149.86 171.45 0)
 			(hide yes)
@@
 			)
 		)
-		(property "Footprint" "Connector_JST:JST_EH_B2B-EH-A_1x02_P2.50mm_Vertical"
+		(property "Footprint" "Connector_JST:JST_EH_S2B-EH_1x02_P2.50mm_Horizontal"
 			(at 354.33 67.31 0)
 			(hide yes)
@@
 			)
 		)
-		(property "Footprint" "Connector_JST:JST_EH_B2B-EH-A_1x02_P2.50mm_Vertical"
+		(property "Footprint" "Connector_JST:JST_EH_S2B-EH_1x02_P2.50mm_Horizontal"
 			(at 344.17 220.98 0)
 			(hide yes)

Commit message: boarded
Parts:
- D3: footprint (none) -> Diode_SMD:D_0805_2012Metric
- J3, J4: footprint Connector_PinHeader_2.54mm:PinHeader_1x05_P2.54mm_Vertical -> Connector_JST:JST_EH_B5B-EH-A_1x05_P2.50mm_Vertical
Connections:
- net +3V3: now also U1.1 (3V3)
- net GPIO36: now also U1.3 (VP_GPIO36); no longer U1.2 (VP_GPIO36)
- net VBAT: no longer R4.1
- net VBAT_FUSED: now also C1.1, C2.1, C3.1, F1.1, R4.1
- no-connect marks 11 -> 10
Other:
- moved on the sheet: F1, Q2
Changed lines of the file:
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@@
 	)
 	(junction
-		(at 359.41 140.97)
+		(at 363.22 140.97)
 		(diameter 0)
 		(color 0 0 0 0)
@@
 	)
 	(no_connect
+		(at 237.49 139.7)
+	)
+	(no_connect
 		(at 273.05 170.18)
 	)
@@
 	)
 	(no_connect
-		(at 237.49 142.24)
-	)
-	(no_connect
-		(at 232.41 137.16)
-	)
-	(no_connect
 		(at 273.05 147.32)
 	)
@@
 	(wire
 		(pts
-			(xy 63.5 49.53) (xy 74.93 49.53)
+			(xy 71.12 49.53) (xy 74.93 49.53)
 		)
 		(stroke
@@
 	(wire
 		(pts
+			(xy 350.52 148.59) (xy 349.25 148.59)
+		)
+		(stroke
+			(width 0)
+			(type default)
+		)
+	)
+	(wire
+		(pts
 			(xy 331.47 119.38) (xy 327.66 119.38)
 		)
@@
 	(wire
 		(pts
-			(xy 349.25 140.97) (xy 359.41 140.97)
+			(xy 349.25 140.97) (xy 381 140.97)
 		)
 		(stroke
@@
 	(wire
 		(pts
-			(xy 64.77 151.13) (xy 74.93 151.13)
+			(xy 350.52 147.32) (xy 350.52 148.59)
 		)
 		(stroke
@@
 	(wire
 		(pts
-			(xy 359.41 140.97) (xy 381 140.97)
-		)
-		(stroke
-			(width 0)
-			(type default)
-		)
-	)
-	(wire
-		(pts
 			(xy 303.53 60.96) (xy 303.53 63.5)
 		)
@@
 	(wire
 		(pts
+			(xy 232.41 129.54) (xy 213.36 129.54)
+		)
+		(stroke
+			(width 0)
+			(type default)
+		)
+	)
+	(wire
+		(pts
 			(xy 195.58 93.98) (xy 195.58 137.16)
 		)
@@
 	(wire
 		(pts
-			(xy 349.25 148.59) (xy 351.79 148.59)
+			(xy 350.52 147.32) (xy 355.6 147.32)
 		)
 		(stroke
@@
 	(wire
 		(pts
+			(xy 213.36 129.54) (xy 213.36 115.57)
+		)
+		(stroke
+			(width 0)
+			(type default)
+		)
+	)
+	(wire
+		(pts
 			(xy 201.93 45.72) (xy 189.23 45.72)
 		)
@@
 	(wire
 		(pts
-			(xy 226.06 139.7) (xy 237.49 139.7)
+			(xy 226.06 142.24) (xy 237.49 142.24)
+		)
+		(stroke
+			(width 0)
+			(type default)
+		)
+	)
+	(wire
+		(pts
+			(xy 232.41 137.16) (xy 232.41 129.54)
 		)
 		(stroke
@@
 	(wire
 		(pts
-			(xy 359.41 154.94) (xy 345.44 154.94)
+			(xy 363.22 154.94) (xy 345.44 154.94)
 		)
 		(stroke
@@
 	(wire
 		(pts
-			(xy 226.06 85.09) (xy 226.06 139.7)
+			(xy 226.06 85.09) (xy 226.06 142.24)
 		)
 		(stroke
@@
 	(wire
 		(pts
-			(xy 53.34 49.53) (xy 55.88 49.53)
+			(xy 53.34 49.53) (xy 63.5 49.53)
 		)
 		(stroke
@@
 	(wire
 		(pts
+			(xy 213.36 115.57) (xy 137.16 115.57)
+		)
+		(stroke
+			(width 0)
+			(type default)
+		)
+	)
+	(wire
+		(pts
 			(xy 200.66 48.26) (xy 189.23 48.26)
 		)
@@
 	(wire
 		(pts
-			(xy 359.41 140.97) (xy 359.41 143.51)
+			(xy 363.22 140.97) (xy 363.22 142.24)
 		)
 		(stroke
@@
 	(wire
 		(pts
-			(xy 336.55 200.66) (xy 346.71 200.66)
+			(xy 336.55 200.66) (xy 345.44 200.66)
 		)
 		(stroke
@@
 	(wire
 		(pts
+			(xy 59.69 151.13) (xy 74.93 151.13)
+		)
+		(stroke
+			(width 0)
+			(type default)
+		)
+	)
+	(wire
+		(pts
 			(xy 82.55 151.13) (xy 92.71 151.13)
 		)
@@
 	(wire
 		(pts
-			(xy 359.41 154.94) (xy 359.41 153.67)
+			(xy 363.22 154.94) (xy 363.22 152.4)
 		)
 		(stroke
@@
 	)
 	(label "GPIO36"
-		(at 229.87 139.7 0)
+		(at 234.95 142.24 180)
 		(effects
 			(font
 				(size 1.27 1.27)
 			)
-			(justify left bottom)
+			(justify right bottom)
 		)
 	)
@@
 		)
 	)
-	(label "GPIO27"
-		(at 228.6 161.29 0)
+	(label "VBAT_FUSED"
+		(at 104.14 49.53 0)
 		(effects
 			(font
@@
 		)
 	)
-	(label "+3V3"
-		(at 166.37 72.39 0)
+	(label "GPIO27"
+		(at 228.6 161.29 0)
 		(effects
 			(font
@@
 		)
 	)
-	(label "VBAT"
-		(at 64.77 151.13 0)
+	(label "+3V3"
+		(at 166.37 72.39 0)
 		(effects
 			(font
@@
 		)
 	)
+	(label "VBAT_FUSED"
+		(at 59.69 151.13 0)
+		(effects
+			(font
+				(size 1.27 1.27)
+			)
+			(justify left bottom)
+		)
+	)
 	(label "GPIO14"
 		(at 231.14 165.1 0)
@@
 	)
 	(label "LIMIT_PWR"
-		(at 346.71 200.66 0)
+		(at 345.44 200.66 0)
 		(effects
 			(font
@@
 			)
 		)
-		(property "Footprint" "Connector_PinHeader_2.54mm:PinHeader_1x05_P2.54mm_Vertical"
+		(property "Footprint" "Connector_JST:JST_EH_B5B-EH-A_1x05_P2.50mm_Vertical"
 			(at 259.08 44.45 0)
 			(hide yes)
@@
 	(symbol
 		(lib_id "Transistor_FET:Q_NMOS_GSD")
-		(at 356.87 148.59 0)
+		(at 360.68 147.32 0)
 		(unit 1)
 		(body_style 1)
@@
 		(dnp no)
 		(property "Reference" "Q2"
-			(at 362.077 147.4216 0)
+			(at 365.887 146.1516 0)
 			(show_name no)
 			(do_not_autoplace no)
@@
 		)
 		(property "Value" "30N06L"
-			(at 362.077 149.733 0)
+			(at 365.887 148.463 0)
 			(show_name no)
 			(do_not_autoplace no)
@@
 		)
 		(property "Footprint" "Package_TO_SOT_THT:TO-220-3_Horizontal_TabUp"
-			(at 356.87 148.59 0)
+			(at 360.68 147.32 0)
 			(hide yes)
 			(show_name no)
@@
 		)
 		(property "Datasheet" ""
-			(at 356.87 148.59 0)
+			(at 360.68 147.32 0)
 			(show_name no)
 			(do_not_autoplace no)
@@
 			)
 		)
-		(property "Description" ""
-			(at 356.87 148.59 0)
+		(property "Description" "N-MOSFET transistor, gate/source/drain"
+			(at 367.792 138.938 0)
 			(show_name no)
 			(do_not_autoplace no)
@@
 			)
 		)
-		(property "Footprint" ""
+		(property "Footprint" "Diode_SMD:D_0805_2012Metric"
 			(at 161.29 165.1 0)
 			(hide yes)
@@
 			)
 		)
-		(property "Description" ""
-			(at 363.22 165.1 0)
+		(property "Description" "P-MOSFET transistor, gate/source/drain"
+			(at 363.22 171.45 0)
 			(show_name no)
 			(do_not_autoplace no)
@@
 	(symbol
 		(lib_id "Device:Fuse")
-		(at 59.69 49.53 270)
+		(at 67.31 49.53 270)
 		(unit 1)
 		(body_style 1)
@@
 		(dnp no)
 		(property "Reference" "F1"
-			(at 59.69 44.5262 90)
+			(at 67.31 44.5262 90)
 			(show_name no)
 			(do_not_autoplace no)
@@
 		)
 		(property "Value" "8A"
-			(at 59.69 46.8376 90)
+			(at 67.31 46.8376 90)
 			(show_name no)
 			(do_not_autoplace no)
@@
 		)
 		(property "Footprint" "Fuse:Fuseholder_Cylinder-5x20mm_Schurter_0031_8201_Horizontal_Open"
-			(at 59.69 49.53 0)
+			(at 67.31 49.53 0)
 			(hide yes)
 			(show_name no)
@@
 		)
 		(property "Datasheet" ""
-			(at 59.69 49.53 0)
+			(at 67.31 49.53 0)
 			(show_name no)
 			(do_not_autoplace no)
@@
 		)
 		(property "Description" ""
-			(at 59.69 49.53 0)
+			(at 67.31 49.53 0)
 			(show_name no)
 			(do_not_autoplace no)
@@
 			)
 		)
-		(property "Footprint" "Connector_PinHeader_2.54mm:PinHeader_1x05_P2.54mm_Vertical"
+		(property "Footprint" "Connector_JST:JST_EH_B5B-EH-A_1x05_P2.50mm_Vertical"
 			(at 220.98 44.45 0)
 			(hide yes)
